File: syncro-mainboard/accessory.kicad_sch (KiCad schematic)
At the start: 16 parts, among them J5 USB_A, J6 USB_A, J7 USB_A, U10 ECMF02-2AMX6, U11 TPS25200, U8 ECMF02-2AMX6, U9 ECMF02-2AMX6

Commit message: Syncro mainboard rev 2
* Migrate I2C to I2C5 on SOM pins 132/133
* Use correctly reversed LED footprint
* Use updated rear graphics
* Set SOM to be assembled at JLC
Other:
- title: USB Accessory Ports -> Syncro FFB Interceptor
Changed lines of the file:
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@@
 	(paper "USLetter")
 	(title_block
-		(title "USB Accessory Ports")
-		(date "2026-08-25")
-		(rev "1")
+		(title "Syncro FFB Interceptor")
+		(date "2026-10-23")
+		(rev "2")
 		(company "Deadband Inc.")
 	)
