File: syncro-mainboard/debug.kicad_sch (KiCad schematic)
At the start: 39 parts, among them J2 Conn_01x03, J3 Conn_ARM_JTAG_SWD_10, Q1 AO3401A, SW1 RESET, SW2 USB BOOT

Commit message: Syncro mainboard rev 2
* Migrate I2C to I2C5 on SOM pins 132/133
* Use correctly reversed LED footprint
* Use updated rear graphics
* Set SOM to be assembled at JLC
Other:
- title: Debug -> Syncro FFB Interceptor
Changed lines of the file:
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@@
 	(paper "USLetter")
 	(title_block
-		(title "Debug")
-		(date "2026-08-25")
-		(rev "1")
+		(title "Syncro FFB Interceptor")
+		(date "2026-10-23")
+		(rev "2")
 		(company "Deadband Inc.")
 	)
