File: syncro-mainboard/gpio.kicad_sch (KiCad schematic)
At the start: 19 parts, among them J8 MikroBUS, J9 Qwiic

Commit message: Syncro mainboard rev 2
* Migrate I2C to I2C5 on SOM pins 132/133
* Use correctly reversed LED footprint
* Use updated rear graphics
* Set SOM to be assembled at JLC
Other:
- title: User GPIO -> Syncro FFB Interceptor
Changed lines of the file:
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@@
 	(paper "USLetter")
 	(title_block
-		(title "User GPIO")
-		(date "2026-08-25")
-		(rev "1")
+		(title "Syncro FFB Interceptor")
+		(date "2026-10-23")
+		(rev "2")
 		(company "Deadband Inc.")
 	)
