File: syncro-mainboard/syncro-mainboard.kicad_pcb (KiCad board)
At the start: 4 copper layers, 78.5 x 59 mm, 145 parts, among them J1 USB_C_Receptacle_USB2.0_16P, J2 Conn_01x03, J3 Conn_ARM_JTAG_SWD_10, J4 Micro_SD_Card_Det1, J5 USB_A, J6 USB_A, J7 USB_A, J8 MikroBUS, J9 Qwiic, Q1 AO3401A, SW1 RESET, SW2 USB BOOT, SW3 SW_USER, U1 MYC-YF135, U10 ECMF02-2AMX6, U11 TPS25200, U2 TS3USB221ARSER, U3 TS3USB221ARSER, U4 ECMF02-2AMX6, U5 FE1.1s, U6 TPS25200, U7 EMIF06-MSD02N16, U8 ECMF02-2AMX6, U9 ECMF02-2AMX6, Y1 12MHz

Commit message: Correct SMD5050 LED rotation
Parts:
- turned D12 to 180 degrees
Connections:
- D12 pad 1: +3.3V -> /System IO/LED_B_X
- D12 pad 2: +3.3V -> /System IO/LED_R_X
- D12 pad 3: +3.3V -> /System IO/LED_G_X
- D12 pad 4: /System IO/LED_B_X -> +3.3V
- D12 pad 5: /System IO/LED_R_X -> +3.3V
- D12 pad 6: /System IO/LED_G_X -> +3.3V
Changed lines of the file:
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@@
 	(footprint "LED_SMD:LED_RGB_5050-6"
 		(layer "F.Cu")
-		(at 97.7 86.25)
+		(at 97.7 86.25 180)
 		(descr "http://cdn.sparkfun.com/datasheets/Components/LED/5060BRG4.pdf")
 		(tags "RGB LED 5050-6")
 		(property "Reference" "D12"
-			(at 0 -3.5 0)
+			(at 0 -3.5 180)
 			(layer "F.SilkS")
 			(hide yes)
@@
 		)
 		(property "Value" "LED_GRB"
-			(at 0 3.3 0)
+			(at 0 3.3 180)
 			(layer "F.Fab")
 			(hide yes)
@@
 		)
 		(property "Datasheet" ""
-			(at 0 0 0)
+			(at 0 0 180)
 			(unlocked yes)
 			(layer "F.Fab")
@@
 		)
 		(property "Description" "RGB LED, 6 pin package"
-			(at 0 0 0)
+			(at 0 0 180)
 			(unlocked yes)
 			(layer "F.Fab")
@@
 		)
 		(property "MPN" "TJ-S5050UG2W5TLCBRG-A5"
-			(at 0 0 0)
+			(at 0 0 180)
 			(unlocked yes)
 			(layer "F.Fab")
@@
 		)
 		(property "LCSC" "C440459"
-			(at 0 0 0)
+			(at 0 0 180)
 			(unlocked yes)
 			(layer "F.Fab")
@@
 		(duplicate_pad_numbers_are_jumpers no)
 		(fp_line
+			(start 2.5 2.7)
+			(end -2.5 2.7)
+			(stroke
+				(width 0.12)
+				(type solid)
+			)
+			(layer "F.SilkS")
+		)
+		(fp_line
 			(start -2.5 -2.7)
 			(end 2.5 -2.7)
-			(stroke
-				(width 0.12)
-				(type solid)
-			)
-			(layer "F.SilkS")
-		)
-		(fp_line
-			(start 2.5 2.7)
-			(end -2.5 2.7)
 			(stroke
 				(width 0.12)
@@
 		)
 		(fp_line
+			(start 3.65 2.75)
+			(end 3.65 -2.75)
+			(stroke
+				(width 0.05)
+				(type solid)
+			)
+			(layer "F.CrtYd")
+		)
+		(fp_line
+			(start 3.65 -2.75)
+			(end -3.65 -2.75)
+			(stroke
+				(width 0.05)
+				(type solid)
+			)
+			(layer "F.CrtYd")
+		)
+		(fp_line
+			(start -3.65 2.75)
+			(end 3.65 2.75)
+			(stroke
+				(width 0.05)
+				(type solid)
+			)
+			(layer "F.CrtYd")
+		)
+		(fp_line
 			(start -3.65 -2.75)
 			(end -3.65 2.75)
@@
 		)
 		(fp_line
-			(start -3.65 2.75)
-			(end 3.65 2.75)
-			(stroke
-				(width 0.05)
-				(type solid)
-			)
-			(layer "F.CrtYd")
-		)
-		(fp_line
-			(start 3.65 -2.75)
-			(end -3.65 -2.75)
-			(stroke
-				(width 0.05)
-				(type solid)
-			)
-			(layer "F.CrtYd")
-		)
-		(fp_line
-			(start 3.65 2.75)
-			(end 3.65 -2.75)
-			(stroke
-				(width 0.05)
-				(type solid)
-			)
-			(layer "F.CrtYd")
+			(start 2.5 2.5)
+			(end 2.5 -2.5)
+			(stroke
+				(width 0.1)
+				(type solid)
+			)
+			(layer "F.Fab")
+		)
+		(fp_line
+			(start 2.5 -2.5)
+			(end -2.5 -2.5)
+			(stroke
+				(width 0.1)
+				(type solid)
+			)
+			(layer "F.Fab")
+		)
+		(fp_line
+			(start -2.5 2.5)
+			(end 2.5 2.5)
+			(stroke
+				(width 0.1)
+				(type solid)
+			)
+			(layer "F.Fab")
+		)
+		(fp_line
+			(start -2.5 -1.9)
+			(end -1.9 -2.5)
+			(stroke
+				(width 0.1)
+				(type solid)
+			)
+			(layer "F.Fab")
 		)
 		(fp_line
 			(start -2.5 -2.5)
 			(end -2.5 2.5)
-			(stroke
-				(width 0.1)
-				(type solid)
-			)
-			(layer "F.Fab")
-		)
-		(fp_line
-			(start -2.5 -1.9)
-			(end -1.9 -2.5)
-			(stroke
-				(width 0.1)
-				(type solid)
-			)
-			(layer "F.Fab")
-		)
-		(fp_line
-			(start -2.5 2.5)
-			(end 2.5 2.5)
-			(stroke
-				(width 0.1)
-				(type solid)
-			)
-			(layer "F.Fab")
-		)
-		(fp_line
-			(start 2.5 -2.5)
-			(end -2.5 -2.5)
-			(stroke
-				(width 0.1)
-				(type solid)
-			)
-			(layer "F.Fab")
-		)
-		(fp_line
-			(start 2.5 2.5)
-			(end 2.5 -2.5)
 			(stroke
 				(width 0.1)
@@
 		)
 		(fp_text user "${REFERENCE}"
-			(at 0 0 0)
+			(at 0 0 180)
 			(layer "F.Fab")
 			(effects
@@
 		)
 		(pad "1" smd rect
-			(at -2.4 -1.7 90)
+			(at -2.4 -1.7 270)
+			(size 1.1 2)
+			(layers "F.Cu" "F.Mask" "F.Paste")
+			(net "/System IO/LED_B_X")
+			(pinfunction "BK_1")
+			(pintype "passive")
+		)
+		(pad "2" smd rect
+			(at -2.4 0 270)
+			(size 1.1 2)
+			(layers "F.Cu" "F.Mask" "F.Paste")
+			(net "/System IO/LED_R_X")
+			(pinfunction "RK_2")
+			(pintype "passive")
+		)
+		(pad "3" smd rect
+			(at -2.4 1.7 270)
+			(size 1.1 2)
+			(layers "F.Cu" "F.Mask" "F.Paste")
+			(net "/System IO/LED_G_X")
+			(pinfunction "GK_3")
+			(pintype "passive")
+		)
+		(pad "4" smd rect
+			(at 2.4 1.7 270)
 			(size 1.1 2)
 			(layers "F.Cu" "F.Mask" "F.Paste")
 			(net "+3.3V")
-			(pinfunction "GA_1")
-			(pintype "passive")
-		)
-		(pad "2" smd rect
-			(at -2.4 0 90)
+			(pinfunction "GA_4")
+			(pintype "passive")
+		)
+		(pad "5" smd rect
+			(at 2.4 0 270)
 			(size 1.1 2)
 			(layers "F.Cu" "F.Mask" "F.Paste")
 			(net "+3.3V")
-			(pinfunction "RA_2")
-			(pintype "passive")
-		)
-		(pad "3" smd rect
-			(at -2.4 1.7 90)
+			(pinfunction "RA_5")
+			(pintype "passive")
+		)
+		(pad "6" smd rect
+			(at 2.4 -1.7 270)
 			(size 1.1 2)
 			(layers "F.Cu" "F.Mask" "F.Paste")
 			(net "+3.3V")
-			(pinfunction "BA_3")
-			(pintype "passive")
-		)
-		(pad "4" smd rect
-			(at 2.4 1.7 90)
-			(size 1.1 2)
-			(layers "F.Cu" "F.Mask" "F.Paste")
-			(net "/System IO/LED_B_X")
-			(pinfunction "BK_4")
-			(pintype "passive")
-		)
-		(pad "5" smd rect
-			(at 2.4 0 90)
-			(size 1.1 2)
-			(layers "F.Cu" "F.Mask" "F.Paste")
-			(net "/System IO/LED_R_X")
-			(pinfunction "RK_5")
-			(pintype "passive")
-		)
-		(pad "6" smd rect
-			(at 2.4 -1.7 90)
-			(size 1.1 2)
-			(layers "F.Cu" "F.Mask" "F.Paste")
-			(net "/System IO/LED_G_X")
-			(pinfunction "GK_6")
-			(pintype "passive")
-		)
+			(pinfunction "BA_6")
+			(pintype "passive")
+		)

Commit message: Syncro mainboard rev 2
* Migrate I2C to I2C5 on SOM pins 132/133
* Use correctly reversed LED footprint
* Use updated rear graphics
* Set SOM to be assembled at JLC
Parts:
- removed the REF** at (132.1, 79.8)
- added REF**: Syncro Graphics, dbl-mech:Syncro_Rear_Graphics, F.Cu at (94.8, 77.3)
- added REF**: DBL Logo Line, dbl-mech:DBL_Logo_Line, B.Cu at (149.2, 78.8)
- moved R44 1.00 mm to (154.0, 89.7)
- moved R45 1.00 mm to (154.0, 90.7)
Connections:
- U1 pad 132: unconnected-(U1Spare 75-148-PF3/LTDC_G3-Pad132) -> /STM32MP13 SOM/I2C_SDA
- U1 pad 133: unconnected-(U1Spare 75-148-PH13/LTDC_G2-Pad133) -> /STM32MP13 SOM/I2C_SCL
- U1 pad 93: /STM32MP13 SOM/I2C_SCL -> unconnected-(U1Expansion-PH3/I2C3_SCL-Pad93)
- U1 pad 94: /STM32MP13 SOM/I2C_SDA -> unconnected-(U1Expansion-PH7/I2C3_SDA-Pad94)
Routing:
- net /STM32MP13 SOM/I2C_SDA: track 7.37 -> 42.4 mm, vias 0 -> 2
- net /STM32MP13 SOM/I2C_SCL: track 7.53 -> 42.2 mm, vias 0 -> 2
- net +5V: track 123.4 -> 114.7 mm
- net /Debug/UART4_TX: track 59.9 -> 61.8 mm
- net /STM32MP13 SOM/GPIO_A0: track 66.3 -> 64.6 mm
- net /Debug/UART4_RX: track 67.3 -> 68.6 mm
- net /System IO/CD: track 45.5 -> 44.5 mm
- net /User GPIO/I2C_SCL_X: track 44.7 -> 43.7 mm, vias 3 -> 1
- net /User GPIO/I2C_SDA_X: track 44.3 -> 45.0 mm
- net GND: vias 177 -> 176
Other:
- board text removed: "Deadband Labs"
- board text removed: "Syncro FFB Interceptor"
