File: syncro-mainboard/usb.kicad_sch (KiCad schematic)
At the start: 38 parts, among them J1 USB_C_Receptacle_USB2.0_16P, U2 TS3USB221ARSER, U3 TS3USB221ARSER, U4 ECMF02-2AMX6, U5 FE1.1s, U6 TPS25200, Y1 12MHz

Commit message: Syncro mainboard rev 2
* Migrate I2C to I2C5 on SOM pins 132/133
* Use correctly reversed LED footprint
* Use updated rear graphics
* Set SOM to be assembled at JLC
Other:
- title: USB Mux -> Syncro FFB Interceptor
Changed lines of the file:
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@@
 	(paper "USLetter")
 	(title_block
-		(title "USB Mux")
-		(date "2026-08-25")
-		(rev "1")
+		(title "Syncro FFB Interceptor")
+		(date "2026-10-23")
+		(rev "2")
 		(company "Deadband Inc.")
 	)
